File: electronics/StartStopSwitch_ver3_0/StartStopSwitch_Ver3_0.brd (EAGLE design)
At the start: 58 x 22.5 mm, 3 parts

Commit message: Update StartStopSwitch ver3.0
Parts:
- renumbered U$1 to M1
Connections:
- removed net +5V: M1.21
Routing:
- net BUTTON0: track 17.1 -> 18.3 mm
Other:
- board text added: "RoboCup Soccer Humanoid Team CIT Brains http://www.cit-brains.net/ SUSTAINA StartStopSwitch Ver3.0 Designed by Masato Kubotera on April 10, 2022."
- board text removed: "RoboCup Soccer Humanoid Team CIT Brains http://www.cit-brains.net/ SUSTAINA StartStopSwitch Ver3.0 Designed by Masato Kubotera on April 1, 2022."
Changed lines of the file:
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@@
 <wire x1="20.78" y1="-9.35" x2="20.78" y2="9.35" width="0.254" layer="51"/>
 <wire x1="20.78" y1="9.35" x2="2.08" y2="9.35" width="0.254" layer="51"/>
-<text x="0" y="0" size="1.27" layer="22" ratio="10" rot="MR180" align="center">RoboCup Soccer Humanoid Team
-CIT Brains http://www.cit-brains.net/
+<text x="0" y="0" size="1.27" layer="22" ratio="10" rot="MR180" align="center">RoboCup Soccer Humanoid Team CIT Brains
+http://www.cit-brains.net/
 SUSTAINA StartStopSwitch Ver3.0
-Designed by Masato Kubotera on April 1, 2022.</text>
+Designed by Masato Kubotera on April 10, 2022.</text>
 </plain>
 <attributes>
@@
 <attribute name="NAME" x="-11.43" y="10.16" size="1.27" layer="25" ratio="10" rot="R180" align="center"/>
 </element>
-<element name="U$1" library="Arduino" package="PRO_MICRO_SMD" value="PRO_MICRO_SMD" x="2.54" y="0" smashed="yes" rot="MR270">
+<element name="M1" library="Arduino" package="PRO_MICRO_SMD" value="PRO_MICRO_SMD" x="2.54" y="0" smashed="yes" rot="MR270">
 <attribute name="NAME" x="-16.51" y="0" size="1" layer="26" ratio="10" rot="MR270" align="center"/>
 </element>
@@
 <contactref element="S1" pad="2"/>
 <contactref element="S1" pad="1"/>
-<contactref element="U$1" pad="1"/>
-<wire x1="-17.78" y1="5.08" x2="-13.94" y2="8.92" width="0.254" layer="16"/>
-<wire x1="-13.94" y1="8.92" x2="-11.43" y2="8.92" width="0.254" layer="16"/>
+<contactref element="M1" pad="1"/>
+<wire x1="-15.845" y1="8.92" x2="-17.78" y2="6.985" width="0.254" layer="16"/>
+<wire x1="-17.78" y1="5.08" x2="-17.78" y2="6.985" width="0.254" layer="16"/>
+<wire x1="-15.845" y1="8.92" x2="-11.43" y2="8.92" width="0.254" layer="16"/>
 <wire x1="-9.7438125" y1="5.08" x2="-11.43" y2="6.7661875" width="0.254" layer="16"/>
 <wire x1="-11.43" y1="8.92" x2="-11.43" y2="6.7661875" width="0.254" layer="16"/>
@@
 <contactref element="S2" pad="2"/>
 <contactref element="S2" pad="1"/>
-<contactref element="U$1" pad="2"/>
+<contactref element="M1" pad="2"/>
 <wire x1="-8.4738125" y1="6.35" x2="-8.89" y2="6.7661875" width="0.254" layer="16"/>
 <wire x1="-8.89" y1="8.92" x2="-8.89" y2="6.7661875" width="0.254" layer="16"/>
@@
 <contactref element="S2" pad="3"/>
 <contactref element="S2" pad="4"/>
-<contactref element="U$1" pad="3"/>
-<contactref element="U$1" pad="4"/>
-<contactref element="U$1" pad="23"/>
+<contactref element="M1" pad="3"/>
+<contactref element="M1" pad="4"/>
+<contactref element="M1" pad="23"/>
 <polygon width="0.254" layer="1">
 <vertex x="-31.75" y="12.7"/>
@@
 </polygon>
 </signal>
-<signal name="+5V">
-<contactref element="U$1" pad="21"/>
-</signal>
 <signal name="SCREW_HOLE1">
 <via x="-25" y="0" extent="1-16" drill="3.2" diameter="5.5" locked="yes"/>
@@
 </signals>
 <mfgpreviewcolors>
-<mfgpreviewcolor name="soldermaskcolor" color="0xC8008000"/>
+<mfgpreviewcolor name="soldermaskcolor" color="0xC8000000"/>
 <mfgpreviewcolor name="silkscreencolor" color="0xFFFEFEFE"/>
 <mfgpreviewcolor name="backgroundcolor" color="0xFF282828"/>
