File: electronics/StartStopSwitch_ver3_0/StartStopSwitch_Ver3_0.sch (EAGLE design)
At the start: 3 parts

Commit message: Update StartStopSwitch ver3.0
Parts:
- renumbered U$1 to M1
Connections:
- removed net +5V: M1.VCC
Changed lines of the file:
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@@
 <part name="SUPPLY1" library="supply2" library_urn="urn:adsk.eagle:library:372" deviceset="AGND" device=""/>
 <part name="SUPPLY2" library="supply2" library_urn="urn:adsk.eagle:library:372" deviceset="AGND" device=""/>
-<part name="U$1" library="Arduino" deviceset="PRO_MICRO_SMD" device=""/>
-<part name="P+1" library="supply1" library_urn="urn:adsk.eagle:library:371" deviceset="+5V" device=""/>
+<part name="M1" library="Arduino" deviceset="PRO_MICRO_SMD" device=""/>
 <part name="SUPPLY3" library="supply2" library_urn="urn:adsk.eagle:library:372" deviceset="AGND" device=""/>
 <part name="SUPPLY4" library="supply2" library_urn="urn:adsk.eagle:library:372" deviceset="AGND" device=""/>
@@
 <attribute name="VALUE" x="53.213" y="-23.495" size="1.778" layer="96"/>
 </instance>
-<instance part="U$1" gate="G$1" x="-10.16" y="-10.16" smashed="yes">
+<instance part="M1" gate="G$1" x="-10.16" y="-10.16" smashed="yes">
 <attribute name="NAME" x="-10.16" y="12.7" size="1.27" layer="95" ratio="10" align="center"/>
-</instance>
-<instance part="P+1" gate="1" x="7.62" y="10.16" smashed="yes">
-<attribute name="VALUE" x="5.08" y="5.08" size="1.778" layer="96" rot="R90"/>
 </instance>
 <instance part="SUPPLY3" gate="G$1" x="-27.94" y="-27.94" smashed="yes">
 <attribute name="VALUE" x="-30.607" y="-31.115" size="1.778" layer="96"/>
 </instance>
-<instance part="SUPPLY4" gate="G$1" x="10.16" y="-27.94" smashed="yes">
-<attribute name="VALUE" x="7.493" y="-31.115" size="1.778" layer="96"/>
+<instance part="SUPPLY4" gate="G$1" x="7.62" y="-27.94" smashed="yes">
+<attribute name="VALUE" x="4.953" y="-31.115" size="1.778" layer="96"/>
 </instance>
 </instances>
@@
 </segment>
 <segment>
-<pinref part="U$1" gate="G$1" pin="1/TX"/>
+<pinref part="M1" gate="G$1" pin="1/TX"/>
 <wire x1="-25.4" y1="5.08" x2="-27.94" y2="5.08" width="0.1524" layer="91"/>
 <label x="-27.94" y="5.08" size="1.778" layer="95" rot="R180"/>
@@
 </segment>
 <segment>
-<pinref part="U$1" gate="G$1" pin="0/RX"/>
+<pinref part="M1" gate="G$1" pin="0/RX"/>
 <wire x1="-25.4" y1="2.54" x2="-27.94" y2="2.54" width="0.1524" layer="91"/>
 <label x="-27.94" y="2.54" size="1.778" layer="95" rot="R180"/>
@@
 <segment>
 <wire x1="-27.94" y1="-25.4" x2="-27.94" y2="-2.54" width="0.1524" layer="91"/>
-<pinref part="U$1" gate="G$1" pin="GND_1"/>
+<pinref part="M1" gate="G$1" pin="GND_1"/>
 <wire x1="-27.94" y1="-2.54" x2="-27.94" y2="0" width="0.1524" layer="91"/>
 <wire x1="-27.94" y1="0" x2="-25.4" y2="0" width="0.1524" layer="91"/>
-<pinref part="U$1" gate="G$1" pin="GND_2"/>
+<pinref part="M1" gate="G$1" pin="GND_2"/>
 <wire x1="-25.4" y1="-2.54" x2="-27.94" y2="-2.54" width="0.1524" layer="91"/>
 <junction x="-27.94" y="-2.54"/>
@@
 </segment>
 <segment>
-<pinref part="U$1" gate="G$1" pin="GND_3"/>
-<wire x1="5.08" y1="2.54" x2="10.16" y2="2.54" width="0.1524" layer="91"/>
-<wire x1="10.16" y1="2.54" x2="10.16" y2="-25.4" width="0.1524" layer="91"/>
+<pinref part="M1" gate="G$1" pin="GND_3"/>
+<wire x1="5.08" y1="2.54" x2="7.62" y2="2.54" width="0.1524" layer="91"/>
+<wire x1="7.62" y1="2.54" x2="7.62" y2="-25.4" width="0.1524" layer="91"/>
 <pinref part="SUPPLY4" gate="G$1" pin="AGND"/>
 </segment>
 </net>
-<net name="+5V" class="0">
-<segment>
-<pinref part="U$1" gate="G$1" pin="VCC"/>
-<wire x1="5.08" y1="-2.54" x2="7.62" y2="-2.54" width="0.1524" layer="91"/>
-<wire x1="7.62" y1="-2.54" x2="7.62" y2="7.62" width="0.1524" layer="91"/>
-<pinref part="P+1" gate="1" pin="+5V"/>
-</segment>
-</net>
