File: electronics/MainBoard_ver2_2/MainBoard_ver2_2.sch (EAGLE design)
At the start: 76 parts, among them IC1 LTC1480, IC2 LTC1480, IC3 LTC1480, IC4 LTC1480, IC5 LTC4412, M1 FT4232H_MINI_MODULE, Q1 SQM40P10-40L_GE3, Q2 SQM40P10-40L_GE3, Q3 SQM40P10-40L_GE3, Q4 SQM40P10-40L_GE3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

Commit message: Update MainBoard ver2.2
Parts:
- added LED5, LED6: (no value), led:LEDSML0603
- added R22: 1k, rcl:R-US_R0603
- added R23: 2k, rcl:R-US_R0603
- CH1, CH2: value XT60PT-M -> XT60PW-M; device AMASS_XT60:XT60PT-M -> AMASS_XT60:XT60PW-M
- IC1, IC2, IC3, IC4: value LTC1480 -> ADM3078E; device LTC1480:LTC1480 -> ADM3078E:ADM3078E
- R13, R14: value 2k -> 1k
- R15: value 470k -> 2k
- R16: value 10k -> 2k
- R17: value 10k -> 470k
- R18: value 2k -> 10k
- R19: value 8.66k -> 10k
- R20: value 1k -> 2k
- R21: value 2k -> 8.66k
- renumbered C17 to C16
Connections:
- removed net VBUS_TO_VCC: M1.VBUS, M1.VCC
- new net +UB: M1.VBUS, M1.VCC, R13.2
- new net LED_3V3: LED2.A, R14.1
- new net LED_UB: LED1.A, R13.1
- net +3V3: now also R14.2
- net AGND: now also LED1.C, LED2.C
- net A_DIODE_DCDC: now also R21.2; no longer R19.2
- net A_FUSE_BATT: now also R16.2; no longer R14.2
- net A_FUSE_DCDC: now also R23.2; no longer R21.2
- net A_FUSE_PWR: now also R15.2; no longer R13.2
- net A_FUSE_SERVO: now also R20.2; no longer R18.2
- net B_LOAD_CPU: now also R19.1; no longer R17.1
- net B_LOAD_SERVO: now also R18.1; no longer R16.1
- net FB_DCDC: now also R21.1, R22.2; no longer R19.1, R20.2
- net GND: now also LED5.C, LED6.C, R22.1; no longer LED1.C, LED2.C, R20.1
- net INPUT_PWR: now also R18.2, R19.2; no longer R15.2, R16.2
- net LED_BATT: now also LED4.A, R16.1; no longer LED2.A, R14.1
- net LED_DCDCOUT: now also LED6.A, R23.1; no longer LED4.A, R21.1
- net LED_PWR: now also LED3.A, R15.1; no longer LED1.A, R13.1
- net LED_SERVO: now also LED5.A, R20.1; no longer LED3.A, R18.1
- net LTC4412_STAT: now also R17.1; no longer R15.1
Other:
- note added: "Conversion from USB to 4-port RS485"
- note added: "State LEDｓ"
- note added: "Termination resistors"
- note added: "UART to RS485"
- note added: "USB to UART"
- moved on the sheet: C1, C2, C3, C4, IC1, IC2, IC3, IC4, LED1, LED2, LED3, LED4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
