File: electronics/EN715_ExpansionBoard_ver1_0/EN715_ExpansionBoard_ver1_0.brd (EAGLE design)
At the start: 87 x 50 mm, 34 parts, among them IC1 FE1.1S, M1 MPU9250_MODULE

Commit message: Update ExpansionBoard_ver1_0
Parts:
- added CH4: S4B-XH-A, JST-XH:S4B-XH-A
- added JP1, JP2, JP3, JP4, JP5, JP6, JP7, JP8: SHORTLAND, Shortland:SHORTLAND
- moved CH2 23.2 mm to (3.49, 15.8)
- moved CH3 7.94 mm to (16.8, 15.8)
- moved FL2 3.22 mm to (-10.2, 6.48)
- moved D3 2.90 mm to (-11.7, 6.48)
- moved D4 2.90 mm to (-13.7, 6.48)
- moved USB2 2.86 mm to (-11.7, 25.0)
- moved M1 2.77 mm to (-20.5, -1.27)
- moved D5 2.59 mm to (-29.2, 6.48)
- moved D6 2.59 mm to (-31.1, 6.48)
- moved FL3 2.59 mm to (-27.3, 6.48)
- moved USB3 2.54 mm to (-29.2, 25.0)
- moved CH1 0.09 mm to (38.7, -4.40)
Connections:
- net EN715_I2S0_LRCK_LS renamed EN715_I2S0_FS
- net EN715_I2S0_SCLK_LS renamed EN715_I2S0_SCLK
- net EN715_I2S0_SDIN_LS renamed EN715_I2S0_DIN
- net EN715_I2S0_SDOUT_LS renamed EN715_I2S0_DOUT
- net EN715_SPI1_CS1_LS renamed EN715_SPI1_CS1
- removed net EN715_ID_I2C_SCL: CH1.12
- removed net EN715_ID_I2C_SDA: CH1.10
- removed net EN715_SPI1_CS0_LS: CH1.17, M1.6
- removed net EN715_SPI1_MISO_LS: CH1.13, M1.5
- removed net EN715_SPI1_MOSI_LS: CH1.15, M1.4
- removed net EN715_SPI1_SCK_LS: CH1.11, M1.3
- removed net N$1: CH2.3
- removed net N$2: CH2.4
- removed net USB-HUB_3_D+: IC1.7
- removed net USB-HUB_3_D-: IC1.6
- new net EN715_I2C0_SCL: CH1.12, CH3.4, JP2.2
- new net EN715_I2C0_SDA: CH1.10, CH3.3, JP4.2
- new net EN715_SPI1_CS0: CH1.17, JP7.2
- new net EN715_SPI1_MISO: CH1.13, JP5.2
- new net EN715_SPI1_MOSI: CH1.15, JP3.2
- new net EN715_SPI1_SCK: CH1.11, JP1.2
- new net MPU9250_AD0/SD0: JP5.1, JP6.1, M1.5
- new net MPU9250_CS: JP7.1, JP8.1, M1.6
- new net MPU9250_SCL/SCLK: JP1.1, JP2.1, M1.3
- new net MPU9250_SDA/SDI: JP3.1, JP4.1, M1.4
- net +3V3: now also CH4.2, JP8.2
- net AGND: now also CH4.1, JP6.2
- net EN715_I2C1_SCL: now also CH4.4
- net EN715_I2C1_SDA: now also CH4.3
- net EN715_UART2_RXD_3V3: now also CH2.4; no longer CH3.4
- net EN715_UART2_TXD_3V3: now also CH2.3; no longer CH3.3
Routing:
- net +3V3: track 0.00 -> 120.0 mm
- net EN715_I2C0_SCL: track 0.00 -> 86.8 mm
- net +5V: track 0.00 -> 79.0 mm, vias 0 -> 4
- net MPU9250_CS: track 0.00 -> 62.8 mm
- net EN715_UART2_TXD_3V3: track 0.00 -> 61.1 mm
- net EN715_I2C0_SDA: track 0.00 -> 59.8 mm, vias 0 -> 1
- net MPU9250_AD0/SD0: track 0.00 -> 54.8 mm
- net EN715_UART2_RXD_3V3: track 0.00 -> 54.3 mm
- net MPU9250_SCL/SCLK: track 0.00 -> 54.3 mm
- net MPU9250_SDA/SDI: track 0.00 -> 53.7 mm
- net USB-HUB_1_D-: track 0.00 -> 45.1 mm
- net USB-HUB_1_D+: track 0.00 -> 40.5 mm
- net USB_IN_D-: track 0.00 -> 38.9 mm
- net USB_IN_D+: track 0.00 -> 38.2 mm
- net EN715_I2C1_SDA: track 0.00 -> 37.6 mm
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Other:
- board text added: "3V3"
- board text added: "Connect MPU9250 to"
- board text added: "GND"
- board text added: "I2C #0 /dev/i2c-0"
- board text added: "I2C #1 /dev/i2c-8"
- board text added: "I2C>"
- board text added: "MPU9250 Module"
- board text added: "Port #1"
- board text added: "Port #2"
- board text added: "RXD"
- board text added: "RoboCup Soccer Humanoid Team CIT Brains http://www.cit-brains.net/"
- board text added: "SCL"
- board text added: "SDA"
- board text added: "SPI>"
- board text added: "SUSTAINA EN715 ExpansionBoard ver1.0 Designed by Masato Kubotera on April 12, 2022."
- board text added: "TXD"
- board text added: "UART #2 /dev/ttyS0"
- board text added: "USB HUB Port #1"
- board text added: "USB HUB Port #2"
- board text added: "X"
- board text added: "Y"
- board text added: "Z"
- board text removed: "Port1"
- board text removed: "Port2"
- board text removed: "^UART"
- board text removed: "^USB Port 1"
- board text removed: "^USB Port 2"
