File: electronics/EN715_ExpansionBoard_ver1_0/EN715_ExpansionBoard_ver1_0.sch (EAGLE design)
At the start: 34 parts, among them IC1 FE1.1S, M1 MPU9250_MODULE

Commit message: Update ExpansionBoard_ver1_0
Parts:
- added CH4: S4B-XH-A, JST-XH:S4B-XH-A
- added JP1, JP2, JP3, JP4, JP5, JP6, JP7, JP8: SHORTLAND, Shortland:SHORTLAND
Connections:
- net EN715_I2S0_LRCK_LS renamed EN715_I2S0_FS
- net EN715_I2S0_SCLK_LS renamed EN715_I2S0_SCLK
- net EN715_I2S0_SDIN_LS renamed EN715_I2S0_DIN
- net EN715_I2S0_SDOUT_LS renamed EN715_I2S0_DOUT
- net EN715_SPI1_CS1_LS renamed EN715_SPI1_CS1
- removed net EN715_ID_I2C_SCL: CH1.12
- removed net EN715_ID_I2C_SDA: CH1.10
- removed net EN715_SPI1_CS0_LS: CH1.17, M1.CS
- removed net EN715_SPI1_MISO_LS: CH1.13, M1.AD0/SD0
- removed net EN715_SPI1_MOSI_LS: CH1.15, M1.SDA/SDI
- removed net EN715_SPI1_SCK_LS: CH1.11, M1.SCL/SCLK
- removed net N$1: CH2.3
- removed net N$2: CH2.4
- removed net USB-HUB_3_D+: IC1.DP3
- removed net USB-HUB_3_D-: IC1.DM3
- new net EN715_I2C0_SCL: CH1.12, CH3.4, JP2.2
- new net EN715_I2C0_SDA: CH1.10, CH3.3, JP4.2
- new net EN715_SPI1_CS0: CH1.17, JP7.2
- new net EN715_SPI1_MISO: CH1.13, JP5.2
- new net EN715_SPI1_MOSI: CH1.15, JP3.2
- new net EN715_SPI1_SCK: CH1.11, JP1.2
- new net MPU9250_AD0/SD0: JP5.1, JP6.1, M1.AD0/SD0
- new net MPU9250_CS: JP7.1, JP8.1, M1.CS
- new net MPU9250_SCL/SCLK: JP1.1, JP2.1, M1.SCL/SCLK
- new net MPU9250_SDA/SDI: JP3.1, JP4.1, M1.SDA/SDI
- net +3V3: now also CH4.2, JP8.2
- net AGND: now also CH4.1, JP6.2
- net EN715_I2C1_SCL: now also CH4.4
- net EN715_I2C1_SDA: now also CH4.3
- net EN715_UART2_RXD_3V3: now also CH2.4; no longer CH3.4
- net EN715_UART2_TXD_3V3: now also CH2.3; no longer CH3.3
- net USB-HUB_1_D+: now also USB2.D+; no longer USB2.A_D+
- net USB-HUB_1_D-: now also USB2.D-; no longer USB2.A_D-
- net USB-HUB_2_D+: now also USB3.D+; no longer USB3.A_D+
- net USB-HUB_2_D-: now also USB3.D-; no longer USB3.A_D-
Other:
- note added: "EN715 20-Pin GPIO"
- note added: "I2C0"
- note added: "I2C1"
- note added: "MPU9250"
- note added: "UART2"
- note removed: "EN715"
- moved on the sheet: CH1, CH2, CH3, D1, D2, F1, FL1, LED1, M1, R1, USB1
