File: electronics/EN715_ExpansionBoard_ver1_1/EN715_ExpansionBoard_ver1_1.brd (EAGLE design)
At the start: 87 x 50 mm, 50 parts, among them IC1 FE1.1S, M1 MPU9250_MODULE

Commit message: Fine-tuned ExpantionBoard Ver1.1 for ordering
Other:
- board text added: "SUSTAINA EN715 ExpansionBoard ver1.1 Designed by Masato Kubotera on April 26, 2022."
- board text removed: "SUSTAINA EN715 ExpansionBoard ver1.1 Designed by Masato Kubotera on April 25, 2022."
Changed lines of the file:
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@@
 <drawing>
 <settings>
-<setting alwaysvectorfont="no"/>
+<setting alwaysvectorfont="yes"/>
 <setting verticaltext="up"/>
 </settings>
@@
  http://www.cit-brains.net/</text>
 <text x="0" y="8.89" size="1.778" layer="21" ratio="10" align="center">SUSTAINA EN715 ExpansionBoard ver1.1
-Designed by Masato Kubotera on April 25, 2022.</text>
+Designed by Masato Kubotera on April 26, 2022.</text>
 <text x="-16.92275" y="-12.3825" size="1.27" layer="22" ratio="10" rot="MR0" align="center">MPU9250 Module</text>
 <text x="32.8295" y="-10.16" size="1" layer="22" ratio="10" rot="MR270" align="center-right">I2C&gt;</text>
@@
 </element>
 <element name="C5" library="rcl" library_urn="urn:adsk.eagle:library:334" package="C0603" package3d_urn="urn:adsk.eagle:package:23616/2" value="22p" x="-26.4795" y="-7.747" smashed="yes" rot="MR90">
-<attribute name="NAME" x="-24.7015" y="-7.747" size="1" layer="26" ratio="10" rot="MR270" align="center"/>
+<attribute name="NAME" x="-25.2095" y="-7.747" size="1" layer="26" ratio="10" rot="MR270" align="center"/>
 <attribute name="POPULARITY" value="37" x="-26.4795" y="-50.927" size="1.778" layer="28" rot="MR90" display="off"/>
 <attribute name="SPICEPREFIX" value="C" x="-26.4795" y="-50.927" size="1.778" layer="28" rot="MR90" display="off"/>
@@
 <wire x1="-41.1070625" y1="-24.13" x2="-36.068" y2="-24.13" width="0.254" layer="16"/>
 <wire x1="-36.068" y1="-24.13" x2="-36.0592" y2="-24.1212" width="0.254" layer="16"/>
-<wire x1="-32.075" y1="11.02" x2="-32.075" y2="17.9782" width="0.254" layer="16"/>
-<wire x1="-32.1018" y1="17.9782" x2="-13.081" y2="17.9782" width="0.254" layer="16"/>
+<wire x1="-32.075" y1="17.9782" x2="-13.081" y2="17.9782" width="0.254" layer="16"/>
 <wire x1="-13.081" y1="17.9782" x2="6.025" y2="17.9782" width="0.254" layer="16"/>
 <wire x1="25.075" y1="15.82735" x2="25.075" y2="11.02" width="0.254" layer="16"/>
@@
 <wire x1="6.025" y1="17.9782" x2="6.025" y2="11.02" width="0.254" layer="16"/>
 <wire x1="6.025" y1="17.9782" x2="22.92415" y2="17.9782" width="0.254" layer="16"/>
-<wire x1="-35.72415" y1="17.9782" x2="-32.075" y2="17.9782" width="0.254" layer="16"/>
+<wire x1="-35.72415" y1="17.9782" x2="-32.1018" y2="17.9782" width="0.254" layer="16"/>
+<wire x1="-32.1018" y1="17.9782" x2="-32.075" y2="17.9782" width="0.254" layer="16"/>
 <wire x1="-42.6847" y1="-2.98561875" x2="-42.672" y2="-2.97291875" width="0.254" layer="16"/>
 <wire x1="-42.6847" y1="-2.98561875" x2="-42.6847" y2="11.01765" width="0.254" layer="16"/>
@@
 <wire x1="-40.132" y1="-7.366" x2="-40.6608" y2="-7.8948" width="0.254" layer="16"/>
 <wire x1="-40.968025" y1="-9.525" x2="-42.6847" y2="-9.525" width="0.254" layer="16"/>
-<wire x1="-32.1018" y1="17.9782" x2="-32.075" y2="11.02" width="0" layer="19" extent="16-16"/>
+<wire x1="-32.075" y1="11.02" x2="-32.075" y2="17.9514" width="0.254" layer="16"/>
+<wire x1="-32.075" y1="17.9514" x2="-32.1018" y2="17.9782" width="0.254" layer="16"/>
 </signal>
 <signal name="USB-HUB_1_D-" class="1">
@@
 <wire x1="-30.734" y1="-18.7465" x2="-30.734" y2="-19.304" width="0.254" layer="16"/>
 <wire x1="-32.551" y1="-22.225" x2="-30.734" y2="-22.225" width="0.254" layer="16"/>
-<via x="-30.734" y="-19.3265" extent="1-16" drill="0.3048"/>
-<via x="-30.734" y="-22.2475" extent="1-16" drill="0.3048"/>
-<wire x1="-30.734" y1="-19.3265" x2="-30.734" y2="-22.2475" width="0.254" layer="1"/>
-<wire x1="-30.734" y1="-22.2475" x2="-30.734" y2="-22.225" width="0" layer="19" extent="16-16"/>
-<wire x1="-30.734" y1="-19.304" x2="-30.734" y2="-19.3265" width="0" layer="19" extent="16-16"/>
+<via x="-30.734" y="-19.304" extent="1-16" drill="0.3048"/>
+<via x="-30.734" y="-22.225" extent="1-16" drill="0.3048"/>
+<wire x1="-30.734" y1="-19.304" x2="-30.734" y2="-22.225" width="0.254" layer="1"/>
 </signal>
 <signal name="VD33" class="2">
@@
 <contactref element="USB3" pad="MH1"/>
 <contactref element="USB3" pad="MH2"/>
-<wire x1="-9.525" y1="5.715" x2="-8.4907" y2="5.715" width="0.254" layer="16"/>
-<wire x1="-8.509" y1="5.715" x2="-7.9375" y2="5.715" width="0.254" layer="16"/>
-<wire x1="-7.9375" y1="5.715" x2="-7.62" y2="5.802" width="0.254" layer="16"/>
 <wire x1="-9.525" y1="5.715" x2="-11.1125" y2="5.715" width="0.254" layer="16"/>
 <wire x1="-9.525" y1="5.715" x2="-9.525" y2="5.677" width="0.254" layer="16"/>
@@
 <wire x1="-15.925" y1="8.94" x2="-15.925" y2="14.72" width="0.254" layer="16"/>
 <wire x1="-11.1125" y1="5.715" x2="-11.43" y2="5.677" width="0.254" layer="16"/>
-<wire x1="-8.4907" y1="5.715" x2="-8.4907" y2="8.128" width="0.254" layer="16"/>
+<wire x1="-8.4907" y1="8.128" x2="-8.4907" y2="5.715" width="0.254" layer="16"/>
 <wire x1="-8.4907" y1="8.128" x2="-7.4813" y2="9.017" width="0.254" layer="16"/>
 <wire x1="-7.4813" y1="12.244175" x2="-6.846975" y2="12.8785" width="0.254" layer="16"/>
@@
 <wire x1="-4.9665" y1="12.8785" x2="-6.846975" y2="12.8785" width="0.254" layer="16"/>
 <wire x1="-7.4813" y1="9.017" x2="-7.4813" y2="12.244175" width="0.254" layer="16"/>
-<wire x1="-9.525" y1="5.677" x2="-8.509" y2="5.715" width="0" layer="19" extent="16-16"/>
+<wire x1="-9.525" y1="5.677" x2="-9.487" y2="5.715" width="0.254" layer="16"/>
+<wire x1="-9.487" y1="5.715" x2="-8.4907" y2="5.715" width="0.254" layer="16"/>
+<wire x1="-8.4907" y1="5.715" x2="-7.707" y2="5.715" width="0.254" layer="16"/>
+<wire x1="-7.707" y1="5.715" x2="-7.62" y2="5.802" width="0.254" layer="16"/>
 </signal>
 <signal name="EN715_5V" class="2">
